File: 5-26/jyot.kicad_pcb (KiCad board)
At the start: 2 copper layers, 45.9 x 45.9 mm, 8 parts, among them J1 Conn_01x02, Q1 BC547

Commit message: Add files via upload
Parts:
- moved D1 7.73 mm to (82.3, 119.7)
Routing:
- net Net-(D1-K): track 21.3 -> 13.4 mm
- net Net-(D1-A): track 22.7 -> 15.2 mm
Changed lines of the file:
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@@
 	(footprint "LED_THT:LED_D3.0mm_Horizontal_O6.35mm_Z10.0mm"
 		(layer "F.Cu")
-		(at 81.77 111.934861 180)
+		(at 82.27 119.65 180)
 		(descr "LED, diameter 3.0mm, horizontal offset 6.35mm, z-position of LED center 10.0mm, 2 pins, generated by kicad-footprint-generator")
 		(tags "LED")
@@
 		)
 		(point
-			(at 80.5 101.784861)
+			(at 81 109.5)
 			(size 2)
 			(layer "F.Fab")
 		)
 		(point
-			(at 80.5 111.934861)
+			(at 81 119.65)
 			(size 2)
 			(layer "F.Fab")
@@
 		(embedded_fonts no)
 	)
+	(gr_line
+		(start 56.5 99)
+		(end 104.5 99)
+		(stroke
+			(width 0.2)
+			(type default)
+		)
+		(layer "F.Cu")
+	)
+	(gr_line
+		(start 56.5 153.5)
+		(end 56.5 99)
+		(stroke
+			(width 0.2)
+			(type default)
+		)
+		(layer "F.Cu")
+	)
+	(gr_line
+		(start 104.5 99)
+		(end 104.5 153.5)
+		(stroke
+			(width 0.2)
+			(type default)
+		)
+		(layer "F.Cu")
+	)
 	(gr_circle
 		(center 80.5 129.5)
@@
 	)
 	(segment
-		(start 79.23 121.81)
-		(end 70.145 130.895)
-		(width 0.2)
-		(layer "F.Cu")
-		(net "Net-(D1-A)")
-	)
-	(segment
-		(start 79.23 111.934861)
-		(end 79.23 121.81)
-		(width 0.2)
-		(layer "F.Cu")
-		(net "Net-(D1-A)")
-	)
-	(segment
-		(start 83 113.164861)
-		(end 81.77 111.934861)
-		(width 0.2)
-		(layer "B.Cu")
-		(net "Net-(D1-K)")
-	)
-	(segment
-		(start 83 132.73)
-		(end 83 113.164861)
-		(width 0.2)
-		(layer "B.Cu")
-		(net "Net-(D1-K)")
+		(start 64.92 137.27)
+		(end 64.92 138.73)
+		(width 0.2)
+		(layer "F.Cu")
+		(net "+9V")
+	)
+	(segment
+		(start 64.92 138.73)
+		(end 71.96 145.77)
+		(width 0.2)
+		(layer "F.Cu")
+		(net "+9V")
+	)
+	(segment
+		(start 65.065 137.125)
+		(end 64.92 137.27)
+		(width 0.2)
+		(layer "F.Cu")
+		(net "+9V")
+	)
+	(segment
+		(start 65.065 130.895)
+		(end 65.065 137.125)
+		(width 0.2)
+		(layer "F.Cu")
+		(net "+9V")
 	)
 	(segment
@@
 	)
 	(segment
-		(start 64.92 137.27)
-		(end 64.92 138.73)
-		(width 0.2)
-		(layer "F.Cu")
-		(net "+9V")
-	)
-	(segment
-		(start 64.92 138.73)
-		(end 71.96 145.77)
-		(width 0.2)
-		(layer "F.Cu")
-		(net "+9V")
-	)
-	(segment
-		(start 65.065 137.125)
-		(end 64.92 137.27)
-		(width 0.2)
-		(layer "F.Cu")
-		(net "+9V")
-	)
-	(segment
-		(start 65.065 130.895)
-		(end 65.065 137.125)
-		(width 0.2)
-		(layer "F.Cu")
-		(net "+9V")
+		(start 79.73 121.31)
+		(end 79.73 119.65)
+		(width 0.2)
+		(layer "F.Cu")
+		(net "Net-(D1-A)")
+	)
+	(segment
+		(start 70.145 130.895)
+		(end 79.73 121.31)
+		(width 0.2)
+		(layer "F.Cu")
+		(net "Net-(D1-A)")
 	)
 	(segment
@@
 		(net "Net-(Q1-B)")
 	)
+	(segment
+		(start 82.27 132)
+		(end 83 132.73)
+		(width 0.2)
+		(layer "B.Cu")
+		(net "Net-(D1-K)")
+	)
+	(segment
+		(start 82.27 119.65)
+		(end 82.27 132)
+		(width 0.2)
+		(layer "B.Cu")
+		(net "Net-(D1-K)")
+	)
 	(embedded_fonts no)
